File: pca9544a_pcb.sch (EAGLE design)
At the start: 37 parts, among them IC1 PCA9544ABS, X6 TSW-102-02-S-S-RA, X7 TSW-102-02-S-S-RA, X8 TSW-102-02-S-S-RA, X9 TSW-102-02-S-S-RA

Commit message: gerber out
Parts:
- GIT1: value adf3d9e -> b5c31e5
Changed lines of the file:
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@@
 <parts>
 <part name="FRAME1" library="frames" deviceset="A4L-LOC" device=""/>
-<part name="GIT1" library="git-revision" deviceset="GIT-REVISION" device="_1.2" value="adf3d9e"/>
+<part name="GIT1" library="git-revision" deviceset="GIT-REVISION" device="_1.2" value="b5c31e5"/>
 <part name="IC1" library="mylib" deviceset="PCA9544A" device="BS"/>
 <part name="R1" library="mylib" deviceset="R-US-*" device="-1608" technology="10K"/>

Commit message: gerber out
Parts:
- GIT1: value b5c31e5 -> dcc5f2d
Changed lines of the file:
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@@
 <parts>
 <part name="FRAME1" library="frames" deviceset="A4L-LOC" device=""/>
-<part name="GIT1" library="git-revision" deviceset="GIT-REVISION" device="_1.2" value="b5c31e5"/>
+<part name="GIT1" library="git-revision" deviceset="GIT-REVISION" device="_1.2" value="dcc5f2d"/>
 <part name="IC1" library="mylib" deviceset="PCA9544A" device="BS"/>
 <part name="R1" library="mylib" deviceset="R-US-*" device="-1608" technology="10K"/>

Commit message: gerber out
Parts:
- GIT1: value dcc5f2d -> 4eef362
Changed lines of the file:
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@@
 <parts>
 <part name="FRAME1" library="frames" deviceset="A4L-LOC" device=""/>
-<part name="GIT1" library="git-revision" deviceset="GIT-REVISION" device="_1.2" value="dcc5f2d"/>
+<part name="GIT1" library="git-revision" deviceset="GIT-REVISION" device="_1.2" value="4eef362"/>
 <part name="IC1" library="mylib" deviceset="PCA9544A" device="BS"/>
 <part name="R1" library="mylib" deviceset="R-US-*" device="-1608" technology="10K"/>
